Commit message: Added changes to operate with U2D2 convertor
Signed-off-by: Meet Gandhi <meet.gandhi@einfochips.com>

File: turtlebot3_manipulation_description/ros2_control/turtlebot3_manipulation_system.ros2_control.xacro (robot description, xacro)
@@ -23,5 +23,5 @@
             <plugin>turtlebot3_manipulation_hardware/TurtleBot3ManipulationSystemHardware</plugin>
             <param name="opencr_id">200</param>
-            <param name="opencr_usb_port">/dev/ttyACM0</param>
+            <param name="opencr_usb_port">/dev/ttyUSB0</param>
             <param name="opencr_baud_rate">1000000</param>
             <param name="dxl_joints_profile_acceleration">100</param>
@@ -32,74 +32,4 @@
         </hardware>
       </xacro:unless>
-      <joint name="${prefix}wheel_left_joint">
-        <command_interface name="velocity">
-          <param name="min">-24.5</param>
-          <param name="max">24.5</param>
-        </command_interface>
-        <state_interface name="position">
-          <param name="initial_value">0.0</param>
-        </state_interface>
-        <state_interface name="velocity">
-          <param name="initial_value">0.0</param>
-        </state_interface>
-      </joint>
-      <joint name="${prefix}wheel_right_joint">
-        <command_interface name="velocity">
-          <param name="min">-24.5</param>
-          <param name="max">24.5</param>
-        </command_interface>
-        <state_interface name="position">
-          <param name="initial_value">0.0</param>
-        </state_interface>
-        <state_interface name="velocity">
-          <param name="initial_value">0.0</param>
-        </state_interface>
-      </joint>
-      <sensor name="imu">
-        <state_interface name="orientation.x">
-          <param name="initial_value">0.0</param>
-        </state_interface>
-        <state_interface name="orientation.y">
-          <param name="initial_value">0.0</param>
-        </state_interface>
-        <state_interface name="orientation.z">
-          <param name="initial_value">0.0</param>
-        </state_interface>
-        <state_interface name="orientation.w">
-          <param name="initial_value">0.0</param>
-        </state_interface>
-        <state_interface name="angular_velocity.x">
-          <param name="initial_value">0.0</param>
-        </state_interface>
-        <state_interface name="angular_velocity.y">
-          <param name="initial_value">0.0</param>
-        </state_interface>
-        <state_interface name="angular_velocity.z">
-          <param name="initial_value">0.0</param>
-        </state_interface>
-        <state_interface name="linear_acceleration.x">
-          <param name="initial_value">0.0</param>
-        </state_interface>
-        <state_interface name="linear_acceleration.y">
-          <param name="initial_value">0.0</param>
-        </state_interface>
-        <state_interface name="linear_acceleration.z">
-          <param name="initial_value">0.0</param>
-        </state_interface>
-      </sensor>
-      <sensor name="battery">
-        <state_interface name="voltage">
-          <param name="initial_value">0.0</param>
-        </state_interface>
-        <state_interface name="percentage">
-          <param name="initial_value">0.0</param>
-        </state_interface>
-        <state_interface name="design_capacity">
-          <param name="initial_value">0.0</param>
-        </state_interface>
-        <state_interface name="present">
-          <param name="initial_value">0.0</param>
-        </state_interface>
-      </sensor>
       <joint name="${prefix}joint1">
         <command_interface name="position">
